File: pcb/I2cBrushlessMotors.sch (KiCad schematic (older format))
At the start: 56 parts, among them J1 Conn_01x03, J2 Conn_01x06, J3 Header, J4 Socket, J5 Conn_01x03, Q1 Q_PMOS_GSD, Q10 Q_PMOS_GSD, Q11 Q_NMOS_GSD, Q12 Q_NMOS_GSD, Q13 Q_PMOS_GSD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

Commit message: Apply vertical connector
Parts:
- J1, J5: footprint Connector_Molex:Molex_PicoBlade_53047-0310_1x03_P1.25mm_Vertical -> footprints:Molex_1x03_P1.25mm_Vertical
Changed lines of the file:
@@
 F 0 "J1" H 1418 1617 50  0000 C CNN
 F 1 "Conn_01x03" H 1418 1526 50  0000 C CNN
-F 2 "Connector_Molex:Molex_PicoBlade_53047-0310_1x03_P1.25mm_Vertical" H 1500 1300 50  0001 C CNN
+F 2 "footprints:Molex_1x03_P1.25mm_Vertical" H 1500 1300 50  0001 C CNN
 F 3 "~" H 1500 1300 50  0001 C CNN
 	1    1500 1300
@@
 F 0 "J5" H 1418 2217 50  0000 C CNN
 F 1 "Conn_01x03" H 1418 2126 50  0000 C CNN
-F 2 "Connector_Molex:Molex_PicoBlade_53047-0310_1x03_P1.25mm_Vertical" H 1500 1900 50  0001 C CNN
+F 2 "footprints:Molex_1x03_P1.25mm_Vertical" H 1500 1900 50  0001 C CNN
 F 3 "~" H 1500 1900 50  0001 C CNN
 	1    1500 1900
@@
 $EndComp
 $Comp
-L power:+3.3V #PWR?
+L power:+3.3V #PWR0110
 U 1 1 5EF33477
 P 2150 4650
-F 0 "#PWR?" H 2150 4500 50  0001 C CNN
+F 0 "#PWR0110" H 2150 4500 50  0001 C CNN
 F 1 "+3.3V" H 2165 4823 50  0000 C CNN
 F 2 "" H 2150 4650 50  0001 C CNN
